File: hardware/destinationWeatherStation_v4-5/destinationWeatherStation_v4-5.kicad_sch (KiCad schematic)
At the start: 35 parts, among them J1 S2B-PH-SM4, J2 MEM2061, J3 STEMMA_QT, Q1 IRLML6244TRPBF, Q2 IRLML6244TRPBF, Q3 DMP2035UVTQ-7, Q4 DMP2035UVTQ-7, SW1 SS-12F44-G5, SW2 PTS647SM38SMTR2LFS, U1 XIAO RP2040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

Commit message: fixing for final version
Parts:
- removed Q3: DMP2035UVTQ-7, lib_fp:SOT23-6P95_280X100L40X37N, symbol lib_sch:PMOS
- removed SW2 (x3): PTS647SM38SMTR2LFS, lib_fp:SW_4.5x4.5, symbol lib_sch:PTS645SK50SMTR92LFS
- added Q3: DMP2035UVTQ-7, lib_fp:SOT23-6P95_280X100L40X37N, symbol lib_sch:PMOS_DGS
- added SW3, SW4, SW5: PTS647SM38SMTR2LFS, lib_fp:SW_4.5x4.5, symbol lib_sch:PTS645SK50SMTR92LFS
- C1: MPN (none) -> KGM15CR51A106MT; mpn KGM15CR51A106KT -> (none); populate 1 -> (none)
- C2, C3, C4: MPN (none) -> KGM15AR51H104KT; mpn KGM15AR51H104KT -> (none); populate 1 -> (none)
- H1, H2, H3, H4: populate 0 -> (none)
- J1: MPN (none) -> S2B-PH-SM4-TB(LF)(SN); mpn S2B-PH-SM4-TB(LF)(SN) -> (none); populate 1 -> (none)
- J2: MPN (none) -> MEM2061-01-188-00-A; mpn MEM2061-01-188-00-A -> (none); populate 1 -> (none)
- J3: MPN (none) -> SM04B-SRSS-TB; mpn SM04B-SRSS-TB -> (none); populate 1 -> (none)
- Q1, Q2: MPN (none) -> IRLML6244TRPBF; mpn IRLML6244TRPBF -> (none); populate 1 -> (none)
- Q4: MPN (none) -> DMP2035UVTQ-7; mpn DMP2035UVTQ-7 -> (none); populate 1 -> (none)
- R1, R10, R2, R3, R4, R5, R6, R7, R8, R9: MPN (none) -> CRCW060310K0JNEB; mpn CRCW060310K0JNEB -> (none); populate 1 -> (none)
- R11, R12: MPN (none) -> CRCW06030000Z0EA; mpn CRCW06030000Z0EA -> (none); populate 1 -> (none)
- SW1: value SS-12F44-G5 -> OS102011MS2QN1; footprint lib_fp:SS-12D07-VG_GA_PA -> lib_fp:OS102011MS2QN1; MPN (none) -> OS102011MS2QN1; mpn SS-12D07-VG 4 NS GA PA -> (none); populate 0 -> (none)
- SW2: MPN (none) -> PTS 647 SM38 SMTR2 LFS; mpn PTS 647 SM38 SMTR2 LFS -> (none); populate 1 -> (none)
- U1: MPN (none) -> RP2040; mpn XIAO RP2040 -> (none); populate 0 -> (none)
- U2: MPN (none) -> BME280; mpn BME280 -> (none); populate 1 -> (none)
- U3: MPN (none) -> HS96L03W2C03; mpn HS96L03W2C03 -> (none); populate 0 -> (none)
Connections:
- net +3V3: now also SW3.1, SW3.2, SW4.1, SW4.2, SW5.1, SW5.2
- net SW3: now also SW3.3, SW3.4
- net SW4: now also SW4.3, SW4.4
- net SW5: now also SW5.3, SW5.4
- net VCC: now also Q3.4
- net at J1.2 (Pin_2), Q1.1, Q2.3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: now also Q3.3
- net at Q1.3, Q2.1, Q4.3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: now also Q3.1, Q3.2, Q3.5, Q3.6
Other:
- moved on the sheet: U3
