File: hardware/destinationWeatherStation_v4-5/destinationWeatherStation_v4-5.kicad_sch (KiCad schematic)
At the start: 35 parts, among them J1 S2B-PH-SM4, J2 MEM2061, J3 STEMMA_QT, Q1 IRLML6244TRPBF, Q2 IRLML6244TRPBF, Q3 DMP2035UVTQ-7, Q4 DMP2035UVTQ-7, SW1 OS102011MS2QN1, SW2 PTS647SM38SMTR2LFS, SW3 PTS647SM38SMTR2LFS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

Commit message: changes
Parts:
- C1: JLCPCB PN (none) -> C1691
- C2, C3, C4: JLCPCB PN (none) -> C1590
- J1: JLCPCB PN (none) -> C295747
- J2: JLCPCB PN (none) -> C5151738
- J3: JLCPCB PN (none) -> C160404
- Q1, Q2: JLCPCB PN (none) -> C5123965
- Q3, Q4: JLCPCB PN (none) -> C5126680
- R1, R10, R2, R3, R4, R5, R6, R7, R8, R9: JLCPCB PN (none) -> C1511834
- R11, R12: JLCPCB PN (none) -> C844915
- SW1: JLCPCB PN (none) -> C221829; now not fitted; now left out of the parts list
- SW2, SW3, SW4, SW5: JLCPCB PN (none) -> C2689502
- U1: JLCPCB PN (none) -> N/A; now not fitted; now left out of the parts list
- U2: JLCPCB PN (none) -> C92489
- U3: JLCPCB PN (none) -> C5248080; now not fitted; now left out of the parts list

Commit message: fixed resistor placement
Connections:
- net +3V3: now also R11.3 (B), R12.1 (A); no longer R11.1 (A), R12.3 (B)
- net GND: now also R11.1 (A), R12.3 (B); no longer R11.3 (B), R12.1 (A)
Changed lines of the file:
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@@
 		(lib_id "lib_sch:Resistor_Jumper_3_Open")
 		(at 138.43 116.84 0)
+		(mirror y)
 		(unit 1)
 		(exclude_from_sim no)
@@
 		(lib_id "lib_sch:Resistor_Jumper_3_Open")
 		(at 156.21 116.84 0)
+		(mirror y)
 		(unit 1)
 		(exclude_from_sim no)
